Commit message: Add files via upload

File: state_publisher/gazebo/gazebomodel/akari_gazebo.gazebo.xacro (robot description, xacro)
@@ -20,6 +20,16 @@
       </ros>
       <update_rate>20</update_rate>
-      <joint_name>akari_servo_joint</joint_name>
-      <joint_name>akari_head_joint</joint_name>
+      <joint_name>pan</joint_name>
+      <joint_name>tilt</joint_name>
+    </plugin>
+    <plugin name="ground_truth" filename="libgazebo_ros_p3d.so">
+      <robotNamespace>akari_xacro</robotNamespace>
+      <frameName>map</frameName>
+      <body_name>base_footprint</body_name>
+      <ros>
+        <namespace>/odometry</namespace>
+        <remapping>odom:=ground_truth</remapping>
+      </ros>
+      <update_rate>10.0</update_rate>
     </plugin>
   </gazebo>

File: state_publisher/gazebo/gazebomodel/akari_gazebo.urdf.xacro (robot description, xacro)
@@ -20,6 +20,6 @@
   </xacro:akarihead>
   <!-- =============== Transmission =============== -->
-  <xacro:akari_trans prefix="servo" interface="VelocityJointInterface" />
-  <xacro:akari_trans prefix="head" interface="VelocityJointInterface" />
+  <xacro:akari_trans prefix="pan" interface="VelocityJointInterface" />
+  <xacro:akari_trans prefix="tilt" interface="VelocityJointInterface" />
   <!-- =============== Gazebo =============== -->
   <ros2_control name="GazeboSystem" type="system">
@@ -33,12 +33,5 @@
       <parameters>$(find state_publisher)/akari_gazebo_model/akari_controll.yaml</parameters>
     </plugin>
-    <plugin name="ground_truth" filename="libgazebo_ros_p3d.so">
-      <robotNamespace>akari_xacro</robotNamespace>
-      <frameName>map</frameName>
-      <bodyName>akari_spawn::base_footprint</bodyName>
-      <topicName>/tracker</topicName>
-      <updateRate>10.0</updateRate>
-    </plugin>
-  </gazebo>
+ </gazebo>
   <xacro:akari_base_gazebo />
   </robot>

File: state_publisher/gazebo/gazebomodel/akari_head.urdf.xacro (robot description, xacro)
@@ -2,5 +2,5 @@
 <robot xmlns:xacro="http://ros.org/wiki/xacro">
   <xacro:macro name="akarihead" params="parent *joint_head">
-    <joint name="akari_head_joint" type="continuous">
+    <joint name="tilt" type="continuous">
       <xacro:insert_block name="joint_head" />
       <axis xyz="1.0 0.0 0.0" />

File: state_publisher/gazebo/gazebomodel/akari_servo.urdf.xacro (robot description, xacro)
@@ -2,5 +2,5 @@
 <robot xmlns:xacro="http://ros.org/wiki/xacro">
   <xacro:macro name="akariservo" params="parent *joint_servo">
-    <joint name="akari_servo_joint" type="continuous">
+    <joint name="pan" type="continuous">
       <xacro:insert_block name="joint_servo" />
       <axis xyz="0.0 0.0 1.0" />

File: state_publisher/gazebo/gazebomodel/akari_transmission.xacro (robot description, xacro)
@@ -2,10 +2,10 @@
 <robot xmlns:xacro="http://ros.org/wiki/xacro">
   <xacro:macro name="akari_trans" params="prefix interface">
-    <transmission name="${prefix}_link">
+    <transmission name="${prefix}">
       <type>transmission_interface/SimpleTransmission</type>
-      <joint name="${prefix}_joint">
+      <joint name="${prefix}">
         <hardwareInterface>${interface}</hardwareInterface>
       </joint>
-      <actuator name="${prefix}_motor">
+      <actuator name="${prefix}">
         <hardwareInterface>${interface}</hardwareInterface>
       </actuator>
