Commit message: add xacro files

File: state_publisher/gazebo/gazebomodel/akari_gazebo.urdf.xacro (robot description, xacro)
@@ -1,86 +1,16 @@
 <?xml version="1.0"?>
-<robot xmlns:xacro="http://ros.org/wiki/xacro">
-    <!-- body -->
-    <link name="base_link">
-        <visual>
-            <origin xyz="0.0 0.0 0.0" rpy="0 0 0"/>
-            <geometry>
-                <mesh filename="package://state_publisher/urdf/akari_body.stl" />
-            </geometry>
-            <material name="gray">
-                <color rgba="0.3 0.3 0.3 1"/>
-            </material>
-        </visual>
-        <collision>
-            <geometry>
-                <box size="0.01 0.01 0.01"/>
-            </geometry>
-        </collision>
-        <inertial>
-          <mass value="50.0"/>
-          <origin xyz="0 0.0 0" rpy="0 0 0"/>
-        <inertia ixx="0.000019" iyy="0.000035" izz="0.000019" ixy="0.000" ixz="0.000" iyz="0.000"/>
-        </inertial>
-    </link>
-    <link name="pan_link">
-        <visual>
-            <origin xyz="0 0.0 0" rpy="0 0 0"/>
-            <geometry>
-                <mesh filename="package://state_publisher/urdf/akari_servo.stl" />
-            </geometry>
-            <material name="gray">
-                <color rgba="0.2 0.2 0.2 1"/>
-            </material>
-        </visual>
-        <collision>
-            <geometry>
-                <box size="0.01 0.01 0.01"/>
-            </geometry>
-        </collision>
-        <inertial>
-          <mass value="0.05"/>
-          <origin xyz="0 0.005 0" rpy="0 0 0"/>
-        <inertia ixx="0.000019" iyy="0.000035" izz="0.000019" ixy="0.000" ixz="0.000" iyz="0.000"/>
-        </inertial>
-    </link>
-    <link name="tilt_link">
-        <visual>
-            <origin xyz="0 0.0 0" rpy="0 0 0"/>
-            <geometry>
-                <mesh filename="package://state_publisher/urdf/akari_head.stl" />
-            </geometry>
-            <material name="gray">
-                <color rgba="0.2 0.2 0.2 1"/>
-            </material>
-        </visual>
-        <collision>
-            <geometry>
-                <box size="0.01 0.01 0.01"/>
-            </geometry>
-        </collision>
-        <inertial>
-          <mass value="0.05"/>
-          <origin xyz="0 0.075 0" rpy="0 0 0"/>
-        <inertia ixx="0.000019" iyy="0.000035" izz="0.000019" ixy="0.000" ixz="0.000" iyz="0.000"/>
-        </inertial>
-    </link>
-    <!-- Robot Footprint -->
-    <link name="base_footprint"/>
-    <joint name="base_joint" type="fixed">
-        <parent link="base_link"/>
-        <child link="base_footprint"/>
-        <origin xyz="0 0 0" rpy="0 0 0"/>
-    </joint>
-    <joint name="servo_joint" type="revolute">
-        <parent link="base_link"/>
-        <child link="pan_link"/>
-        <axis xyz="0.0 0.0 1.0"/>
-        <dynamics damping="1.0"/>
-    </joint>
-    <joint name="head_joint" type="revolute">
-        <parent link="pan_link"/>
-        <child link="tilt_link"/>
-        <axis xyz="1.0 0.0 0.0"/>
-        <dynamics damping="1.0"/>
-    </joint>
+<robot name="akari_xacro" xmlns:xacro="http://ros.org/wiki/xacro">
+  <xacro:include filename="$(find state_publisher)/akari_gazebo_model/akari_body.urdf.xacro"/>
+  <xacro:include filename="$(find state_publisher)/akari_gazebo_model/akari_servo.urdf.xacro"/>
+  <xacro:include filename="$(find state_publisher)/akari_gazebo_model/akari_head.urdf.xacro"/>
+  <link name="base_footprint"/>
+  <xacro:akaribase parent="base_footprint">
+    <origin xyz="0 0 0.005" rpy="0 0 0" />
+  </xacro:akaribase>
+  <xacro:akariservo parent="base_link">
+    <origin xyz="0.0 0.012 0.055" rpy="0 0 0" />
+  </xacro:akariservo>
+  <xacro:akarihead parent="servo_link">
+    <origin xyz="0.0 -0.024 0.020" rpy="0 0 0" />
+  </xacro:akarihead>
 </robot>

Commit message: Add files via upload

File: state_publisher/gazebo/gazebomodel/akari_gazebo.urdf.xacro (robot description, xacro)
@@ -1,8 +1,13 @@
 <?xml version="1.0"?>
 <robot name="akari_xacro" xmlns:xacro="http://ros.org/wiki/xacro">
+  <!-- =============== File include =============== -->
   <xacro:include filename="$(find state_publisher)/akari_gazebo_model/akari_body.urdf.xacro"/>
   <xacro:include filename="$(find state_publisher)/akari_gazebo_model/akari_servo.urdf.xacro"/>
   <xacro:include filename="$(find state_publisher)/akari_gazebo_model/akari_head.urdf.xacro"/>
+  <xacro:include filename="$(find state_publisher)/akari_gazebo_model/akari_transmission.xacro"/>
+  <xacro:include filename="$(find state_publisher)/akari_gazebo_model/akari_gazebo.gazebo.xacro"/>
+  <!-- =============== Base =============== -->
   <link name="base_footprint"/>
+  <!-- =============== Model =============== -->
   <xacro:akaribase parent="base_footprint">
     <origin xyz="0 0 0.005" rpy="0 0 0" />
@@ -12,5 +17,28 @@
   </xacro:akariservo>
   <xacro:akarihead parent="servo_link">
-    <origin xyz="0.0 -0.024 0.020" rpy="0 0 0" />
+    <origin xyz="0.0 -0.024 0.025" rpy="0 0 0" />
   </xacro:akarihead>
-</robot>
+  <!-- =============== Transmission =============== -->
+  <xacro:akari_trans prefix="servo" interface="VelocityJointInterface" />
+  <xacro:akari_trans prefix="head" interface="VelocityJointInterface" />
+  <!-- =============== Gazebo =============== -->
+  <ros2_control name="GazeboSystem" type="system">
+    <hardware>
+      <plugin>gazebo_ros2_control/GazeboSystem</plugin>
+    </hardware>
+  </ros2_control>
+  <gazebo>
+    <plugin name="gazebo_ros_control" filename="libgazebo_ros2_control.so">
+      <robotNamespace>akari_xacro</robotNamespace>
+      <parameters>$(find state_publisher)/akari_gazebo_model/akari_controll.yaml</parameters>
+    </plugin>
+    <plugin name="ground_truth" filename="libgazebo_ros_p3d.so">
+      <robotNamespace>akari_xacro</robotNamespace>
+      <frameName>map</frameName>
+      <bodyName>akari_spawn::base_footprint</bodyName>
+      <topicName>/tracker</topicName>
+      <updateRate>10.0</updateRate>
+    </plugin>
+  </gazebo>
+  <xacro:akari_base_gazebo />
+  </robot>

File: state_publisher/gazebo/gazebomodel/akari_head.urdf.xacro (robot description, xacro)
@@ -2,5 +2,5 @@
 <robot xmlns:xacro="http://ros.org/wiki/xacro">
   <xacro:macro name="akarihead" params="parent *joint_head">
-    <joint name="head_joint" type="continuous">
+    <joint name="akari_head_joint" type="continuous">
       <xacro:insert_block name="joint_head" />
       <axis xyz="1.0 0.0 0.0" />

File: state_publisher/gazebo/gazebomodel/akari_servo.urdf.xacro (robot description, xacro)
@@ -2,5 +2,5 @@
 <robot xmlns:xacro="http://ros.org/wiki/xacro">
   <xacro:macro name="akariservo" params="parent *joint_servo">
-    <joint name="servo_joint" type="continuous">
+    <joint name="akari_servo_joint" type="continuous">
       <xacro:insert_block name="joint_servo" />
       <axis xyz="0.0 0.0 1.0" />

Commit message: Add files via upload

File: state_publisher/gazebo/gazebomodel/akari_gazebo.urdf.xacro (robot description, xacro)
@@ -27,8 +27,24 @@
       <plugin>gazebo_ros2_control/GazeboSystem</plugin>
     </hardware>
+    <joint name="pan">
+        <state_interface name="position">
+          <param name="initial_value">0.0</param>
+        </state_interface>
+      <state_interface name="velocity"/>
+      <state_interface name="effort"/>
+    </joint>
+    <joint name="tilt">
+        <state_interface name="position">
+          <param name="initial_value">0.0</param>
+        </state_interface>
+      <state_interface name="velocity"/>
+      <state_interface name="effort"/>
+    </joint>
   </ros2_control>
   <gazebo>
     <plugin name="gazebo_ros_control" filename="libgazebo_ros2_control.so">
       <robotNamespace>akari_xacro</robotNamespace>
+      <robot_param>robot_description</robot_param>
+      <robot_param_node>robot_state_publisher</robot_param_node>
       <parameters>$(find state_publisher)/akari_gazebo_model/akari_controll.yaml</parameters>
     </plugin>
