Commit message: Update akari.urdf

File: state_publisher/urdf/akari.urdf (robot description, URDF)
Before this commit: robot akari, 4 links, 3 joints
Links:
- link base_link: mass None -> 0.05; geometry collision box size=0.01 0.01 0.01; visual mesh filename=package://state_publisher/urdf/akari_body.stl
- link pan_link: mass None -> 0.05; geometry collision box size=0.01 0.01 0.01; visual mesh filename=package://state_publisher/urdf/akari_servo.stl
- link tilt_link: mass None -> 0.05; geometry collision box size=0.01 0.01 0.01; visual mesh filename=package://state_publisher/urdf/akari_head.stl
Joints:
- removed joint head_joint
- removed joint servo_joint
- added joint pan: type continuous, parent base_link, child pan_link, origin xyz=0.0 0.012 0.055 rpy=0 0 0, axis 0 0 1
- added joint tilt: type continuous, parent pan_link, child tilt_link, origin xyz=0.0 -0.024 0.019 rpy=0 0 0, axis 1 0 0

Commit message: Update akari.urdf

File: state_publisher/urdf/akari.urdf (robot description, URDF)
Before this commit: robot akari_urdf, 4 links, 3 joints
Joints:
- joint pan: limit (none) -> lower=-1.0 upper=1.0 effort=30 velocity=30

Commit message: Update akari.urdf

File: state_publisher/urdf/akari.urdf (robot description, URDF)
Before this commit: robot akari_urdf, 4 links, 3 joints
Joints:
- joint pan: limit lower=-1.0 upper=1.0 effort=30 velocity=30 -> (none)
